Commit message: feat: add ZED camera ROS2 wrapper components and configuration files

File: src/jaka_description/urdf/jaka_zu5.urdf (robot description, URDF)
Before this commit: robot jaka_zu5, 18 links, 17 joints
Links:
- link camera_mount_link: geometry collision box size=0.04 0.08 0.01; visual mesh filename=package://jaka_description/meshes/onrobot_2fg7_meshes/camer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 scale=0.001 0.001 0.001
